Commit message: urdfがrvizに表示されない

File: ros2_navigation_test/urdf/first_robot.urdf (robot description, URDF)
Before this commit: robot rover, 3 links, 2 joints
Links:
- added link camera_link, mass 0.5; visual box size=0.05 0.25 0.1
- added link front_caster; collision sphere radius=0.075; visual sphere radius=0.075
- added link imu_link; collision box size=0.05 0.05 0.05; visual box size=0.05 0.05 0.05
- added link lidar_link, mass 0.5; visual cylinder length=0.05 radius=0.05
- added link wheel_front_left, mass 2; collision cylinder length=0.05 radius=0.075; visual cylinder length=0.05 radius=0.075
Joints:
- added joint camera_joint: type fixed, parent base_link, child camera_link, origin xyz=-0.175 0 0.1 rpy=0 0.0 3.14, axis 0.0 0.0 1.0
- added joint caster_joint: type fixed, parent base_link, child front_caster, origin xyz=-0.15 0.0 0 rpy=0 0 0
- added joint imu_joint: type fixed, parent base_link, child imu_link, origin xyz=0 0 0.075 rpy=0 0 0, axis 0 0 1.0
- added joint lidar_joint: type fixed, parent base_link, child lidar_link, origin xyz=-0.215 0 0.0 rpy=0 0.0 1.57, axis 0.0 0.0 1.0
- added joint wheel_front_left_joint: type continuous, parent base_link, child wheel_front_left, origin xyz=0.125 -0.2 0.0 rpy=1.57 0.0 0.0, axis 0.0 0.0 1.0

Commit message: Rvizとgazeboに表示できるようになった

File: ros2_navigation_test/urdf/first_robot.urdf (robot description, URDF)
Before this commit: robot rover, 8 links, 7 joints
Links:
- link imu_link: mass None -> 0.3
Joints:
- joint base_joint: child base_footprint -> base_link; origin xyz=0.0 0.0 -0.075 rpy=0 0 0 -> xyz=0.0 0.0 0.075 rpy=0 0 0; parent base_link -> base_footprint
